Commit message: Add files via upload

File: mpc_controller/JerbotBeta/urdf/jerbotBeta.urdf (robot description, URDF)
Before this commit: robot jerbotBeta, 9 links, 8 joints
Links:
- removed link foot_pitch_left
- removed link foot_pitch_right
- added link foot_left, mass 0.001; visual sphere radius=0.015
- added link foot_right, mass 0.001; visual sphere radius=0.015
- link base: mass 0.1 -> 0.5; geometry collision mesh filename=../meshes/stl/Part__Feature.002.stl scale=1.0 1.0 1.0; collision mesh filename=../meshes/stl/Part__Feature001.002.stl scale=1.0 1.0 1.0
- link knee_pitch_left: geometry collision mesh filename=../meshes/stl/Part__Feature012.001.stl scale=1.0 1.0 1.0; collision sphere radius=0.015
- link knee_pitch_right: geometry collision mesh filename=../meshes/stl/Part__Feature005.001.stl scale=1.0 1.0 1.0; collision sphere radius=0.015
Joints:
- removed joint foot_pitch_left
- removed joint foot_pitch_right
- added joint foot_left: type fixed, parent knee_pitch_left, child foot_left, origin xyz=0.0044 -0.2311 -0.00113 rpy=1.5708 0 3.14159
- added joint foot_right: type fixed, parent knee_pitch_right, child foot_right, origin xyz=0.0046 0.23103 0.01234 rpy=-1.5708 0 -3.14159
